Commit message: update readme

File: src/wro_robosim/description/wro_car/camera.xacro (robot description, xacro)
@@ -58,8 +58,34 @@
         <parent link="camera_link"/>
         <child link="iris_link"/>
-        <origin xyz="${cam_l/2} 0 ${cam_w*0.75}" rpy="0.0 0.0 0.0"/>
+        <origin xyz="${cam_l/2} 0 ${cam_w*0.75}" rpy="0.0 ${radians(7.5)} 0.0"/>
     </joint>
+     <joint name="camera_optical_joint" type="fixed">
+        <parent link="iris_link"/>
+        <child link="camera_link_optical"/>
+        <origin xyz="0 0 0" rpy="${-pi/2} 0 ${-pi/2}"/>
+    </joint>
+    <link name="camera_link_optical"></link>
     <gazebo reference="iris_link">
         <material>Gazebo/Black</material>
+        <sensor name="camera" type="camera">
+            <pose> 0 0 0 0 0 0 </pose>
+            <visualize>false</visualize>
+            <update_rate>30</update_rate>
+            <camera>
+                <horizontal_fov>${radians(40)}</horizontal_fov>
+                <image>
+                    <format>R8G8B8</format>
+                    <width>640</width>
+                    <height>480</height>
+                </image>
+                <clip>
+                    <near>0.001</near>
+                    <far>3</far>
+                </clip>
+            </camera>
+            <plugin name="camera_controller" filename="libgazebo_ros_camera.so">
+                <frame_name>camera_link_optical</frame_name>
+            </plugin>
+        </sensor>
     </gazebo>
 </robot>

File: src/wro_robosim/description/wro_car/colors.xacro (robot description, xacro)
@@ -1,11 +1,11 @@
 <robot xmlns:xacro="http://www.ros.org/wiki/xacro">
-    <material name="red">
-        <color rgba="${68/255} ${214/255} ${44/255} 1"/>
+    <material name="green">
+        <color rgba="0 1 0 1"/>
     </material>
     <material name="blue">
         <color rgba="0 0 1 1"/>
     </material>
-    <material name="green">
-        <color rgba="${238/255} ${39/255} ${55/255} 1"/>
+    <material name="red">
+        <color rgba="1 0 0 1"/>
     </material>
     <material name="grey">

File: src/wro_robosim/description/wro_car/ros2control.xacro (robot description, xacro)
@@ -13,5 +13,5 @@
         <state_interface name="position"/>
       </joint>
-    <joint name="rear_right_wheel_rotate">
+      <joint name="rear_right_wheel_rotate">
         <command_interface name="velocity">
           <param name="min">-20</param>
@@ -21,5 +21,5 @@
         <state_interface name="position"/>
       </joint>
-    <joint name="rear_left_wheel_rotate">
+      <joint name="rear_left_wheel_rotate">
         <command_interface name="velocity">
           <param name="min">-20</param>
@@ -29,13 +29,13 @@
         <state_interface name="position"/>
       </joint>
-    <joint name="front_right_wheel_rotate">
+      <joint name="front_right_wheel_rotate">
         <state_interface name="position"/>
       </joint>
-    <joint name="front_left_wheel_rotate">
+      <joint name="front_left_wheel_rotate">
         <state_interface name="position"/>
       </joint>
     </ros2_control>
     <gazebo>
-      <plugin filename="libgazebo_ros2_control.so" name="gazebo_ros2_control">
+      <plugin name="gazebo_ros2_control" filename="libgazebo_ros2_control.so" >
         <parameters>$(find wro_robosim)/config/ackermanncontroller.yaml</parameters>
       </plugin>

File: src/wro_robosim/description/wro_obstacle_world/colors.xacro (robot description, xacro)
@@ -1,4 +1,4 @@
 <robot xmlns:xacro="http://www.ros.org/wiki/xacro">
-    <material name="red">
+    <material name="green">
         <color rgba="${68/255} ${214/255} ${44/255} 1"/>
     </material>
@@ -6,5 +6,5 @@
         <color rgba="0 0 1 1"/>
     </material>
-    <material name="green">
+    <material name="red">
         <color rgba="${238/255} ${39/255} ${55/255} 1"/>
     </material>

File: src/wro_robosim/description/wro_obstacle_world/obstacle_mat.urdf.xacro (robot description, xacro)
@@ -2,4 +2,5 @@
 <robot xmlns:xacro="http://www.ros.org/wiki/xacro" name="wro_world">
     <link name="world_base_link"/>
+    <xacro:arg name="data" default="[[0,0,0,0,0,0],[0,0,0,0,0,0],[0,0,0,0,0,0],[0,0,0,0,0,0]]" />
     <xacro:arg name="mat_config" default="[0, 0, 0, 0]"/>
     <!-- sides extension status -->
@@ -21,4 +22,5 @@
     <xacro:include filename="inertials.xacro"/>
     <xacro:include filename="wall.xacro"/>
+    <xacro:include filename="parts.xacro"/>
     <!-- mat link loaded from collada meshfile -->
     <link name="mat_link">
@@ -63,3 +65,68 @@
     <xacro:wall link_name="right_inner_wall" x="${iww/2+rsv}" y="${tsv/2-bsv/2}" l="${ril}" dir="0"/>
     <xacro:wall link_name="left_inner_wall" x="${-iww/2-lsv}" y="${tsv/2-bsv/2}" l="${lil}" dir="0"/>
+    <xacro:property name="section_blocks_data" value="${$(arg data)}" />
+    <!-- placing block in each section -->
+    <xacro:section id="0" blocks_data="${section_blocks_data[0]}">
+        <origin xyz="0.5 -0.5 ${mh}" rpy="0.0 0.0 0.0"/>
+    </xacro:section>
+    <xacro:section id="1" blocks_data="${section_blocks_data[1]}">
+        <origin xyz="0.5 0.5 ${mh}" rpy="0.0 0.0 ${pi/2}"/>
+    </xacro:section>
+    <xacro:section id="2" blocks_data="${section_blocks_data[2]}">
+        <origin xyz="-0.5 0.5 ${mh}" rpy="0.0 0.0 ${pi}"/>
+    </xacro:section>
+    <xacro:section id="3" blocks_data="${section_blocks_data[3]}">
+        <origin xyz="-0.5 -0.5 ${mh}" rpy="0.0 0.0 ${3*pi/2}"/>
+    </xacro:section>
+    <!-- parking area -->
+    <link name="park_wall1">
+        <visual>
+            <geometry>
+                <box size="0.2 0.02 0.1"/>
+            </geometry>
+            <material name="magenta"/>
+        </visual>
+        <collision>
+            <geometry>
+                <box size="0.2 0.02 0.1"/>
+            </geometry>
+            <material name="magenta"/>
+        </collision>
+        <xacro:box_inertia x="0.2" y="0.02" z="0.1">
+            <origin xyz="0.0 0.0 0.0" rpy="0.0 0.0 0.0"/>
+        </xacro:box_inertia>
+    </link>
+    <joint name="park_wall1_joint" type="fixed">
+        <parent link="world_base_link"/>
+        <child link="park_wall1"/>
+        <origin xyz="${0.5+0.9} 0.5 ${0.05+mh}" rpy="0.0 0.0 0.0"/>
+    </joint>
+    <gazebo reference="park_wall1">
+        <material>Gazebo/Purple</material>
+    </gazebo>
+    <link name="park_wall2">
+        <visual>
+            <geometry>
+                <box size="0.2 0.02 0.1"/>
+            </geometry>
+            <material name="magenta"/>
+        </visual>
+        <collision>
+            <geometry>
+                <box size="0.2 0.02 0.1"/>
+            </geometry>
+            <material name="magenta"/>
+        </collision>
+        <xacro:box_inertia x="0.2" y="0.02" z="0.1">
+            <origin xyz="0.0 0.0 0.0" rpy="0.0 0.0 0.0"/>
+        </xacro:box_inertia>
+    </link>
+    <joint name="park_wall2_joint" type="fixed">
+        <parent link="world_base_link"/>
+        <child link="park_wall2"/>
+        <origin xyz="${0.5+0.9} ${0.5-1.5*0.184} ${0.05+mh}" rpy="0.0 0.0 0.0"/>
+    </joint>
+    <gazebo reference="park_wall2">
+        <material>Gazebo/Purple</material>
+    </gazebo>
 </robot>

File: src/wro_robosim/description/wro_obstacle_world/wall.xacro (robot description, xacro)
@@ -10,6 +10,5 @@
                 </geometry>
                 <material name="">
-                    <color rgba="1.0 0.0 0.0 1.0"/>
-                    <texture filename=""/>
+                    <color rgba="0 0.0 0.0 1.0"/>
                 </material>
             </visual>
